Commit message: (DOCS) fixed bash scripts

File: match_slam/description/urdf/drone.urdf.xacro (robot description, xacro)
@@ -29,5 +29,5 @@
       rpy="$(arg lidar_rpy)"
       topic_name="$(arg lidar_topic)"
-      mesh_uri="package://match_slam/description/meshes/livox_mid-360.stl"
+      mesh_uri="package://match_models/sdf/match_drohne/meshes/livox_mid-360.stl"
       mesh_scale="0.001 0.001 0.001" />  <!-- use 0.001 if STL is in millimeters -->
   <!-- Mount Camera -->

File: match_slam/description/urdf/drone_core.xacro (robot description, xacro)
@@ -15,6 +15,6 @@
         <origin xyz="0 0 -0.35" rpy="0 0 3.141592654"/>
         <geometry>
-          <!-- <mesh filename="meshes/Drohnen-Modell.glb" scale="1 1 1"/> -->
-          <mesh filename="package://match_slam/description/meshes/Drohnen-Modell.stl" scale="1 1 1"/>
+          <mesh filename="package://match_models/sdf/match_drohne/meshes/Drohnen-Modell.glb" scale="1 1 1"/>
+          <!-- <mesh filename="package://match_models/sdf/match_drohne/meshes/Match-Drohne.stl" scale="1 1 1"/> -->
         </geometry>
       </visual>

File: match_slam/description/urdf/lidar.xacro (robot description, xacro)
@@ -4,5 +4,5 @@
   <xacro:macro name="lidar_sensor" params="parent_link frame_name xyz rpy
                                    topic_name:=/scan
-                                   mesh_uri:=package://match_slam/description/meshes/livox_mid-360.stl
+                                   mesh_uri:=package://match_models/sdf/match_drohne/meshes/livox_mid-360.stl
                                    mesh_scale:='0.001 0.001 0.001'">
     <!-- LiDAR link + fixed joint to parent -->
