Commit message: Emily wollte das (SLAM Vorbereitung)

File: match_models/sdf/match_drohne_alles/match_drohne_alles.xacro (robot description, xacro)
@@ -86,5 +86,5 @@
     <parent link="front_depth_camera_link"/>
     <child link="front_depth_camera_optical_frame"/>
-    <origin xyz="0 0 0" rpy="-1.57079632679 0 -1.57079632679"/>
+    <origin xyz="0 0 0" rpy="0 0 0"/>
   </joint>
   <link name="top_lidar_link">

Commit message: Ich habe schlimme Schmerzen

File: match_models/sdf/match_drohne_alles/match_drohne_alles.xacro (robot description, xacro)
@@ -115,3 +115,30 @@
     <origin xyz="0 0 0" rpy="0 0 0"/>
   </joint>
+  <link name="mid_360_link">
+    <inertial>
+      <mass value="0.02"/>
+      <origin xyz="0 0 0" rpy="0 0 0"/>
+      <inertia ixx="5e-05" ixy="0.0" ixz="0.0" iyy="5e-05" iyz="0.0" izz="5e-05"/>
+    </inertial>
+    <visual>
+      <origin xyz="0 0 0" rpy="0 0 0"/>
+      <geometry>
+        <cylinder radius="0.05" length="0.06"/>
+      </geometry>
+      <material name="lidar_black">
+        <color rgba="0.05 0.05 0.05 1.0"/>
+      </material>
+    </visual>
+  </link>
+  <joint name="mid_360_joint" type="fixed">
+    <parent link="base_link"/>
+    <child link="mid_360_link"/>
+    <origin xyz="${lidar_offset_x} ${lidar_offset_y} ${lidar_offset_z}" rpy="0 0 0"/>
+  </joint>
+  <link name="mid_360_frame"/>
+  <joint name="mid_360_frame_joint" type="fixed">
+    <parent link="mid_360_link"/>
+    <child link="mid_360_frame"/>
+    <origin xyz="0 0 0" rpy="0 0 0"/>
+  </joint>
 </robot>

Commit message: liest das eigentlich jemand?

File: match_models/sdf/match_drohne_alles/match_drohne_alles.xacro (robot description, xacro)
@@ -42,5 +42,5 @@
     <parent link="base_link"/>
     <child link="front_sensor_mount_link"/>
-    <origin xyz="${front_sensor_offset_x} ${front_sensor_offset_y} ${front_sensor_offset_z}" rpy="0 0 0"/>
+    <origin xyz="0.1 0 -0.08" rpy="0 0.2 0"/>
   </joint>
   <link name="front_rgb_camera_link">

Commit message: Hex hex

File: match_models/sdf/match_drohne_alles/match_drohne_alles.xacro (robot description, xacro)
@@ -42,5 +42,5 @@
     <parent link="base_link"/>
     <child link="front_sensor_mount_link"/>
-    <origin xyz="0.1 0 -0.08" rpy="0 0.2 0"/>
+    <origin xyz="0.10 0 -0.1069" rpy="0 0.2 0"/>
   </joint>
   <link name="front_rgb_camera_link">
@@ -134,5 +134,5 @@
     <parent link="base_link"/>
     <child link="mid_360_link"/>
-    <origin xyz="${lidar_offset_x} ${lidar_offset_y} ${lidar_offset_z}" rpy="0 0 0"/>
+    <origin xyz="0.12 0 0.0537" rpy="0 0.5236 0"/>
   </joint>
   <link name="mid_360_frame"/>
@@ -142,3 +142,9 @@
     <origin xyz="0 0 0" rpy="0 0 0"/>
   </joint>
+  <link name="RGLLidar"/>
+  <joint name="RGLLidar_joint" type="fixed">
+    <parent link="mid_360_link"/>
+    <child link="RGLLidar"/>
+    <origin xyz="0 0 0" rpy="0 0 0"/>
+  </joint>
 </robot>

Commit message: ad astra per aspera

File: match_models/sdf/match_drohne_alles/match_drohne_alles.xacro (robot description, xacro)
@@ -14,10 +14,19 @@
     </inertial>
     <visual>
-      <origin xyz="0 0 0" rpy="0 0 0"/>
+      <origin xyz="0 0 -0.35" rpy="0 0 3.141592654"/>
       <geometry>
-        <cylinder radius="0.15" length="0.05"/>
+        <mesh filename="package://match_models/sdf/match_drohne_alles/meshes/Drohnen-Modell.glb" scale="1 1 1"/>
       </geometry>
-      <material name="grey">
+      <material name="drone_body">
         <color rgba="0.3 0.3 0.3 1.0"/>
+      </material>
+    </visual>
+    <visual>
+      <origin xyz="0 0 -0.06" rpy="0 0 1.570796327"/>
+      <geometry>
+        <mesh filename="package://match_models/sdf/match_drohne_alles/meshes/Marvin.stl" scale="0.1 0.1 0.1"/>
+      </geometry>
+      <material name="marvin">
+        <color rgba="0.8 0.8 0.8 1.0"/>
       </material>
     </visual>
